File: pcb/hamockswing.kicad_sch (KiCad schematic)
At the start: 17 parts

Commit message: stuff
Parts:
- removed C? (x2): C, symbol Device:C
- removed J?: Conn_01x04, symbol Connector_Generic:Conn_01x04
- removed TP? (x4): TestPoint, symbol Connector:TestPoint
- removed U?: ATmega88-20A, Package_QFP:TQFP-32_7x7mm_P0.8mm, symbol MCU_Microchip_ATmega:ATmega88-20A
- removed Y?: Crystal, symbol Device:Crystal
- added D3: LED, LED_SMD:LED_0805_2012Metric, symbol Device:LED
- added J3: Conn_01x03, Connector_PinHeader_2.54mm:PinHeader_1x03_P2.54mm_Horizontal, symbol Connector_Generic:Conn_01x03
- added R3: R, Resistor_SMD:R_0603_1608Metric, symbol Device:R
- added U1: ATmega88-20A, Package_QFP:TQFP-32_7x7mm_P0.8mm, symbol MCU_Microchip_ATmega:ATmega88-20A
- C3: renamed from C?; footprint (none) -> Capacitor_SMD:C_0603_1608Metric
- D1, D2: renamed from D?; footprint (none) -> Diode_SMD:D_SOD-123F
- J1: renamed from J?; footprint (none) -> Connector_PinHeader_2.54mm:PinHeader_1x06_P2.54mm_Horizontal
- J2: renamed from J?; footprint (none) -> Connector_PinHeader_2.54mm:PinHeader_2x03_P2.54mm_Vertical
- Q1: renamed from Q?; footprint (none) -> Package_TO_SOT_SMD:SOT-223
- R1, R2: renamed from R?; footprint (none) -> Resistor_SMD:R_0603_1608Metric
Connections:
- net +5V: now also J3.1 (Pin_1), U1.18 (AVCC), U1.4 (VCC), U1.6 (VCC)
- net ENC A: now also U1.1 (PD3)
- net ENC B: now also U1.32 (PD2)
- net GND: now also D3.1 (K), J3.3 (Pin_3), U1.21 (GND), U1.3 (GND), U1.5 (GND)
- net MISO: now also U1.16 (PB4)
- net MOSI: now also U1.15 (PB3)
- net RST: now also U1.29 (~{RESET}/PC6)
- net SCK: now also U1.17 (PB5)
- net TX: now also J3.2 (Pin_2), U1.31 (PD1)
- net at Q1.1 (G), R2.2: now also U1.26 (PC3)
- new net: D3.2 (A), R3.1
- new net LED: R3.2, U1.27 (PC4)
Other:
- moved on the sheet: C3, D1, D2, Q1, R1, R2

Commit message: stuff
Parts:
- added C1, C2, C4, C5, C?: C, Capacitor_SMD:C_0603_1608Metric, symbol Device:C
- added H1, H2: MountingHole, MountingHole:MountingHole_3.2mm_M3_ISO7380_Pad, symbol Mechanical:MountingHole
Connections:
- net +5V: now also D1.2 (A), D2.1 (K), C1.2, C2.2, C4.2, C5.2; no longer D1.1 (K)
- net GND: now also C1.1, C2.1, C4.1, C5.1; no longer J1.2 (Pin_2)
- net MOTOR-: now reaches D2.2 (A), Q1.2 (D)
- net MOTOR-: now also J1.2 (Pin_2), C?.1; no longer D1.2 (A)
- net MOTOR renamed MOTOR+
- net MOTOR+: now also D1.1 (K), C?.2; no longer D2.1 (K)
Other:
- moved on the sheet: D1, D2

Commit message: kind of works, pcb as delivered to eurocircuits
Parts:
- C1, C2: footprint Capacitor_SMD:C_0603_1608Metric -> Capacitor_SMD:C_0805_2012Metric
- gave numbers to parts that had none: 1
Changed lines of the file:
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@@
   (symbol (lib_id "Device:C") (at 167.64 66.04 180) (unit 1)
     (in_bom yes) (on_board yes) (fields_autoplaced)
-    (property "Reference" "C?" (id 0) (at 171.45 64.7699 0)
+    (property "Reference" "C6" (id 0) (at 171.45 64.7699 0)
       (effects (font (size 1.27 1.27)) (justify right))
     )
@@
       (effects (font (size 1.27 1.27)) (justify right))
     )
-    (property "Footprint" "Capacitor_SMD:C_0603_1608Metric" (id 2) (at 35.8648 72.39 0)
+    (property "Footprint" "Capacitor_SMD:C_0805_2012Metric" (id 2) (at 35.8648 72.39 0)
       (effects (font (size 1.27 1.27)) hide)
     )
@@
   (symbol (lib_id "power:+5V") (at 148.59 57.15 0) (unit 1)
     (in_bom yes) (on_board yes)
-    (property "Reference" "#PWR?" (id 0) (at 148.59 60.96 0)
+    (property "Reference" "#PWR0106" (id 0) (at 148.59 60.96 0)
       (effects (font (size 1.27 1.27)) hide)
     )
@@
       (effects (font (size 1.27 1.27)) (justify right))
     )
-    (property "Footprint" "Capacitor_SMD:C_0603_1608Metric" (id 2) (at 46.0248 72.39 0)
+    (property "Footprint" "Capacitor_SMD:C_0805_2012Metric" (id 2) (at 46.0248 72.39 0)
       (effects (font (size 1.27 1.27)) hide)
     )
@@
     )
     (path "/ae825602-75e7-4d7b-8d8f-11e36175d2b9"
-      (reference "#PWR?") (unit 1) (value "+5V") (footprint "")
+      (reference "#PWR0106") (unit 1) (value "+5V") (footprint "")
     )
     (path "/a990ee4b-bf94-4bcf-95cf-17a4d16384fb"
-      (reference "C1") (unit 1) (value "C") (footprint "Capacitor_SMD:C_0603_1608Metric")
+      (reference "C1") (unit 1) (value "C") (footprint "Capacitor_SMD:C_0805_2012Metric")
     )
     (path "/de114387-3d6a-4aef-ae12-909e43474c19"
-      (reference "C2") (unit 1) (value "C") (footprint "Capacitor_SMD:C_0603_1608Metric")
+      (reference "C2") (unit 1) (value "C") (footprint "Capacitor_SMD:C_0805_2012Metric")
     )
     (path "/cd02993b-3248-416d-a869-0c8c31fa2be1"
@@
     )
     (path "/20a7a9ed-fea3-426d-aed5-a2f224ffaf47"
-      (reference "C?") (unit 1) (value "C") (footprint "Capacitor_SMD:C_0603_1608Metric")
+      (reference "C6") (unit 1) (value "C") (footprint "Capacitor_SMD:C_0603_1608Metric")
     )
     (path "/e37c1a7f-003c-40dd-8a31-67fed4c8d9aa"

Commit message: jerk opt
Parts:
- removed C1, C2: C, Capacitor_SMD:C_0805_2012Metric, symbol Device:C
- removed C4, C5, C6: C, Capacitor_SMD:C_0603_1608Metric, symbol Device:C
- removed H1, H2: MountingHole, MountingHole:MountingHole_3.2mm_M3_ISO7380_Pad, symbol Mechanical:MountingHole
Connections:
- net +5V: now also D1.1 (K), J3.3 (Pin_3); no longer D1.2 (A), D2.1 (K), J3.1 (Pin_1)
- net GND: now also J1.2 (Pin_2), J3.1 (Pin_1); no longer J3.3 (Pin_3)
- net MOTOR+ renamed MOTOR
- net MOTOR: now also D2.1 (K); no longer D1.1 (K)
- net MOTOR-: no longer names the net of D2.2 (A), Q1.2 (D)
- net MOTOR-: now also D1.2 (A); no longer J1.2 (Pin_2)
Other:
- moved on the sheet: D1, D2

Commit message: new
Parts:
- added C1, C2, C6: C, Capacitor_SMD:C_0603_1608Metric, symbol Device:C
- added C4, C5: C, Capacitor_SMD:C_0805_2012Metric, symbol Device:C
- renumbered D2 to D1, D1 to D2
Connections:
- net +5V: now also D1.1 (K), J3.1 (Pin_1), C1.2, C2.2, C4.2, C5.2; no longer J3.3 (Pin_3)
- net GND: now also J3.3 (Pin_3), C1.1, C2.1, C4.1, C5.1; no longer J1.2 (Pin_2), J3.1 (Pin_1)
- net at Q1.1 (G), R2.2: now also U1.13 (PB1); no longer U1.26 (PC3)
- net MOTOR-: now reaches D2.2 (A), Q1.2 (D)
- net MOTOR-: now also J1.2 (Pin_2), C6.1; no longer D1.2 (A)
- net MOTOR renamed MOTOR+
- net MOTOR+: now also D1.2 (A), C6.2; no longer D1.1 (K)
Other:
- moved on the sheet: D1, D2
